Commit message: first commit

File: urdf/gazebo_control.xacro (robot description, xacro)
@@ -1,37 +1,27 @@
 <?xml version="1.0"?>
 <robot xmlns:xacro="http://www.ros.org/wiki/xacro">
-    <xacro:macro name="gazebo_control">
-        <gazebo>
-            <plugin name="gazebo_ros_ackermann_drive" filename="libgazebo_ros_ackermann_drive.so">
-                <update_rate>100.0</update_rate>
-                <!-- Wheel joints (Matching names from mobRob.xacro) -->
-                <front_left_joint>front_left_joint</front_left_joint>
-                <front_right_joint>front_right_joint</front_right_joint>
-                <rear_left_joint>rear_left_joint</rear_left_joint>
-                <rear_right_joint>rear_right_joint</rear_right_joint>
-                <!-- Steering joints (Removed extra steering wheel joint) -->
-                <left_steering_joint>front_left_joint</left_steering_joint>
-                <right_steering_joint>front_right_joint</right_steering_joint>
-                <!-- Steering Constraints -->
-                <max_steer>0.6</max_steer>
-                <max_steering_angle>0.8</max_steering_angle>
-                <!-- Speed Constraints -->
-                <max_speed>5.0</max_speed>
-                <!-- PID Tuning -->
-                <left_steering_pid_gain>10 0 1</left_steering_pid_gain>
-                <left_steering_i_range>0 0</left_steering_i_range>
-                <right_steering_pid_gain>10 0 1</right_steering_pid_gain>
-                <right_steering_i_range>0 0</right_steering_i_range>
-                <linear_velocity_pid_gain>100 0 1</linear_velocity_pid_gain>
-                <linear_velocity_i_range>0 0</linear_velocity_i_range>
-                <!-- Output Publishing -->
-                <publish_odom>true</publish_odom>
-                <publish_odom_tf>true</publish_odom_tf>
-                <publish_wheel_tf>true</publish_wheel_tf>
-                <publish_distance>true</publish_distance>
-                <odometry_frame>odom</odometry_frame>
-                <robot_base_frame>base_link</robot_base_frame>
-            </plugin>
-        </gazebo>
-    </xacro:macro>
+  <gazebo>
+    <plugin name="gazebo_ros_ackermann_drive" filename="libgazebo_ros_ackermann_drive.so">
+      <update_rate>100.0</update_rate>
+      <front_left_joint>front_left_joint</front_left_joint>
+      <front_right_joint>front_right_joint</front_right_joint>
+      <rear_left_joint>rear_left_joint</rear_left_joint>
+      <rear_right_joint>rear_right_joint</rear_right_joint>
+      <max_steer>0.6</max_steer>
+      <max_steering_angle>0.8</max_steering_angle>
+      <max_speed>5.0</max_speed>
+      <publish_odom>true</publish_odom>
+      <publish_odom_tf>true</publish_odom_tf>
+      <publish_wheel_tf>true</publish_wheel_tf>
+      <odometry_frame>odom</odometry_frame>
+      <robot_base_frame>base_link</robot_base_frame>
+      <wheel_separation>0.92</wheel_separation>
+      <wheel_radius>0.22</wheel_radius>
+      <wheel_base>0.9066666666666666</wheel_base>
+      <command_topic>cmd_vel</command_topic>
+      <odometry_topic>odom</odometry_topic>
+      <odometry_frame>odom</odometry_frame>
+      <robot_base_frame>base_link</robot_base_frame>
+    </plugin>
+  </gazebo>
 </robot>
